Commit message: xacro fixed

File: fa_ROS2_ws/src/smart_car/urdf/smartcar.urdf (robot description, URDF)
Before this commit: robot smartcar, 11 links, 10 joints
Links:
- link back_left_wheel_link: mass 0.1 -> 0.5
- link back_right_wheel_link: mass 0.1 -> 0.5
- link base_footprint: mass None -> 1; geometry 
- link base_link: mass 0.1 -> None; geometry 
- link chassis_link: mass 1.0 -> 3.0; geometry visual box size=0.257 0.17 0.021333333333333333
- link front_left_wheel_link: mass 0.1 -> 0.5
- link front_left_wheel_steer_link: mass 0.01 -> 0.1
- link front_right_wheel_link: mass 0.1 -> 0.5
- link front_right_wheel_steer_link: mass 0.01 -> 0.1
Joints:
- joint back_left_wheel_joint: origin xyz=-0.1285 0.0975 0.025 rpy=0 0 0 -> xyz=-0.1285 0.11000000000000001 0.032 rpy=0 0 0
- joint back_right_wheel_joint: origin xyz=-0.1285 -0.0975 0.025 rpy=0 0 0 -> xyz=-0.1285 -0.11000000000000001 0.032 rpy=0 0 0
- joint base_footprint_joint: origin xyz=0 0 -0.032 rpy=0 0 0 -> (none)
- joint chassis_joint: origin xyz=0 0 0 rpy=0 0 0 -> xyz=0 0 0.04
- joint front_left_wheel_steer_joint: limit lower=-0.785 upper=0.785 effort=1000 velocity=100 -> lower=-0.7853981633974483 upper=0.7853981633974483 effort=10 velocity=1; origin xyz=0.1285 0.0975 0.025 rpy=0 0 0 -> xyz=0.1285 0.11000000000000001 0.032 rpy=0 0 0
- joint front_right_wheel_steer_joint: limit lower=-0.785 upper=0.785 effort=1000 velocity=100 -> lower=-0.7853981633974483 upper=0.7853981633974483 effort=10 velocity=1; origin xyz=0.1285 -0.0975 0.025 rpy=0 0 0 -> xyz=0.1285 -0.11000000000000001 0.032 rpy=0 0 0
- joint imu_joint: origin xyz=0 0 0.025 -> xyz=0 0 0.082
- joint lidar_joint: origin xyz=0.1285 0 0.082 -> xyz=0.0985 0 0.082

File: fa_ROS2_ws/src/smart_car/urdf/smartcar.urdf.xacro (robot description, xacro)
@@ -1,156 +1,161 @@
 <?xml version="1.0"?>
-<robot name="smartcar" xmlns:xacro="http://ros.org/wiki/xacro">
-<xacro:property name="wheelbase_length" value = "0.257"/>
-<xacro:property name="wheelbase_width" value = "0.17"/>
-<xacro:property name="wheelbase_height" value = "0.05"/>
-<xacro:property name="wheel_diameter" value="0.064"/>
-<xacro:property name="wheel_width" value="0.025"/>
-<!--inertia property macros-->
-<xacro:macro name="box_inertia" params="m w h d">
-    <inertial>
-        <origin xyz="0 0 0" rpy="0 0 0"/>
-        <mass value="${m}"/>
-        <inertia ixx="${(m/12) * (h*h + d*d)}" ixy="0.0" ixz="0.0" iyy="${(m/12) * (w*w + d*d)}" iyz="0.0" izz="${(m/12) * (w*w + h*h)}"/>
-    </inertial>
-</xacro:macro>
-<xacro:macro name="cylinder_inertia" params="m r h">
-    <inertial>
-      <origin xyz="0 0 0" rpy="0 0 0" />
-      <mass value="${m}"/>
-      <inertia ixx="${(m/12) * (3*r*r + h*h)}" ixy="0" ixz="0" iyy="${(m/12) * (3*r*r + h*h)}" iyz="0" izz="${(m/2) * (r*r)}"/>
-    </inertial>
-  </xacro:macro>
-<!--base-->
-<link name="base_link">
-    <visual>
-        <origin xyz = "0 0 ${wheelbase_height/2}" rpy = "0 0 0"/>
-        <geometry>
-        <box size="${wheelbase_length} ${wheelbase_width} ${wheelbase_height}"/>
-        </geometry>
-    </visual>
-    <collision>
-    <origin xyz = "0 0 ${wheelbase_height/2}" rpy = "0 0 0"/>
-        <geometry>
-        <box size="${wheelbase_length} ${wheelbase_width} ${wheelbase_height}"/>
-        </geometry>
-    </collision>
-    <xacro:box_inertia m="0.1" w="${wheelbase_width}" d="${wheelbase_length}" h="${wheelbase_height}"/>
-</link>
-<link name="base_footprint">
-    <visual>
-        <origin xyz="0 0 0" rpy="0 0 0"/>
-        <geometry>
-            <box size="0.001 0.001 0.001"/>
-        </geometry>
-    </visual>
-</link>
-<joint name="base_footprint_joint" type="fixed">
-    <parent link="base_link"/>
-    <child link="base_footprint"/>
-    <origin xyz="0 0 -${wheel_diameter/2}" rpy="0 0 0"/>
-</joint>
-<link name="chassis_link">
-    <visual>
-        <origin xyz="0 0 ${wheelbase_height/2}" rpy="0 0 0"/>
-        <geometry>
-            <box size="${wheelbase_length} ${wheelbase_width} ${wheelbase_height}"/>
-        </geometry>
-    </visual>
-    <collision>
-        <origin xyz="0 0 ${wheelbase_height/2}" rpy="0 0 0"/>
-        <geometry>
-            <box size="${wheelbase_length} ${wheelbase_width} ${wheelbase_height}"/>
-        </geometry>
-    </collision>
-    <xacro:box_inertia m="1.0" w="${wheelbase_width}" d="${wheelbase_length}" h="${wheelbase_height}"/>
-</link>
-<joint name="chassis_joint" type="fixed">
-    <parent link="base_link"/>
-    <child link="chassis_link"/>
-    <origin xyz="0 0 0" rpy="0 0 0"/>
-</joint>
-<!-- Wheels -->
-<xacro:macro name="wheel" params="prefix x_reflect y_reflect joint_name">
-<link name="${prefix}_link">
-    <visual>
-        <origin xyz="0 0 0" rpy="${pi/2} 0 0"/>
-        <geometry>
-            <cylinder radius="${wheel_diameter/2}" length="${wheel_width}"/>
-        </geometry>
-        <material name="Gray">
-            <color rgba="0.5 0.5 0.5 1.0"/>
-        </material>
-    </visual>
-    <collision>
-        <origin xyz="0 0 0" rpy="${pi/2} 0 0"/>
-        <geometry>
-            <cylinder radius="${wheel_diameter/2}" length="${wheel_width}"/>
-        </geometry>
-    </collision>
-    <xacro:cylinder_inertia m="0.1" r="${wheel_diameter/2}" h="${wheel_width}"/>
-</link>
-<joint name="${joint_name}" type="continuous">
-    <parent link="base_link"/>
-    <child link="${prefix}_link"/>
-    <origin xyz="${-x_reflect * wheelbase_length/2} ${(y_reflect * (wheelbase_width/2 + wheel_width/2))} ${wheelbase_height/2}" rpy="0 0 0"/>
+<robot xmlns:xacro="http://www.ros.org/wiki/xacro" name="smartcar">
+  <!-- ==================== Properties ==================== -->
+  <!-- Dimensions -->
+  <xacro:property name="wheel_diameter" value="0.064" />
+  <xacro:property name="wheel_width" value="0.025" />
+  <xacro:property name="wheelbase_length" value="0.257" />
+  <xacro:property name="wheelbase_width" value="0.17" />
+  <xacro:property name="Lidar_radius" value="0.03" />
+  <!-- Masses and inertial properties -->
+  <xacro:property name="wheel_mass" value="0.5" />
+  <xacro:property name="chassis_mass" value="3.0" />
+  <xacro:property name="chassis_height" value="${wheel_diameter/4}" />
+  <xacro:property name="steer_link_mass" value="0.1" />
+  <xacro:property name="steer_link_size" value="0.01" />
+  <xacro:property name="imu_mass" value="0.05" />
+  <xacro:property name="imu_size" value="0.05" />
+  <xacro:property name="lidar_mass" value="0.05" />
+  <xacro:property name="lidar_height" value="0.05" />
+  <!-- ==================== Wheel Macros ==================== -->
+  <!-- Front wheel with steering -->
+  <xacro:macro name="front_wheel" params="prefix parent x y z">
+    <link name="front_${prefix}_wheel_link">
+      <inertial>
+        <mass value="${wheel_mass}"/>
+        <inertia
+          ixx="${(wheel_mass/12) * (3*(wheel_diameter/2)*(wheel_diameter/2) + wheel_width*wheel_width)}"
+          ixy="0.0"
+          ixz="0.0"
+          iyy="${(wheel_mass/12) * (3*(wheel_diameter/2)*(wheel_diameter/2) + wheel_width*wheel_width)}"
+          iyz="0.0"
+          izz="${(wheel_mass/2) * (wheel_diameter/2)*(wheel_diameter/2)}"/>
+        <origin xyz="0 0 0" rpy="${pi/2} 0 0"/>
+      </inertial>
+      <visual>
+        <origin xyz="0 0 0" rpy="${pi/2} 0 0"/>
+        <geometry>
+          <cylinder radius="${wheel_diameter/2}" length="${wheel_width}"/>
+        </geometry>
+      </visual>
+      <collision>
+        <origin xyz="0 0 0" rpy="${pi/2} 0 0"/>
+        <geometry>
+          <cylinder radius="${wheel_diameter/2}" length="${wheel_width}"/>
+        </geometry>
+      </collision>
+    </link>
+    <link name="front_${prefix}_wheel_steer_link">
+      <visual>
+          <geometry>
+              <box size="0.01 0.01 0.01"/>
+          </geometry>
+          <origin xyz="0 0 0" rpy="0 0 0"/>
+      </visual>
+      <collision>
+          <geometry>
+              <box size="0.01 0.01 0.01"/>
+          </geometry>
+          <origin xyz="0 0 0" rpy="0 0 0"/>
+      </collision>
+      <inertial>
+          <mass value="${steer_link_mass}"/>
+          <origin xyz="0 0 0" rpy="0 0 0"/>
+          <inertia
+            ixx="${(steer_link_mass/6) * (steer_link_size*steer_link_size)}"
+            ixy="0.0"
+            ixz="0.0"
+            iyy="${(steer_link_mass/6) * (steer_link_size*steer_link_size)}"
+            iyz="0.0"
+            izz="${(steer_link_mass/6) * (steer_link_size*steer_link_size)}"/>
+      </inertial>
+  </link>
+    <joint name="front_${prefix}_wheel_steer_joint" type="revolute">
+      <origin xyz="${x} ${y} ${z}" rpy="0 0 0"/>
+      <parent link="${parent}"/>
+      <child link="front_${prefix}_wheel_steer_link"/>
+      <axis xyz="0 0 1"/>
+      <limit lower="-${45 * (pi / 180)}" upper="${45 * (pi / 180)}" effort="10" velocity="1"/>
+  </joint>
+  <joint name="front_${prefix}_wheel_joint" type="continuous">
+    <origin xyz="0 0 0" rpy="0 0 0" />
+    <parent link="front_${prefix}_wheel_steer_link"/>
+    <child link="front_${prefix}_wheel_link"/>
     <axis xyz="0 1 0"/>
 </joint>
-</xacro:macro>
-<!-- Front Wheels with Steering -->
-<xacro:macro name="steering_wheel" params="prefix x_reflect y_reflect steer_joint_name wheel_joint_name">
-<link name="${prefix}_steer_link">
+  </xacro:macro>
+  <!-- Back wheel -->
+  <xacro:macro name="back_wheel" params="prefix parent x y z">
+    <link name="back_${prefix}_wheel_link">
+      <inertial>
+        <mass value="0.5"/>
+        <inertia ixx="0.0001" ixy="0.0" ixz="0.0" iyy="0.0001" iyz="0.0" izz="0.0002"/>
+        <origin xyz="0 0 0" rpy="${pi/2} 0 0"/>
+      </inertial>
+      <visual>
+        <origin xyz="0 0 0" rpy="${pi/2} 0 0"/>
+        <geometry>
+          <cylinder radius="${wheel_diameter/2}" length="${wheel_width}"/>
+        </geometry>
+      </visual>
+      <collision>
+        <origin xyz="0 0 0" rpy="${pi/2} 0 0"/>
+        <geometry>
+          <cylinder radius="${wheel_diameter/2}" length="${wheel_width}"/>
+        </geometry>
+      </collision>
+    </link>
+    <joint name="back_${prefix}_wheel_joint" type="continuous">
+      <parent link="${parent}" />
+      <child link="back_${prefix}_wheel_link"/>
+      <origin xyz="${x} ${y} ${z}" rpy="0 0 0"/>
+      <axis xyz="0 1 0"/>
+    </joint>
+  </xacro:macro>
+  <!-- ==================== Robot Base ==================== -->
+  <!-- Base footprint and chassis -->
+  <link name="base_link">
+  </link>
+  <link name="base_footprint">
+    <inertial>
+      <mass value="1"/>
+      <inertia ixx="0.01" ixy="0.0" ixz="0.0" iyy="0.01" iyz="0.0" izz="0.02"/>
+      <origin xyz="0 0 0"/>
+    </inertial>
+  </link>
+  <joint name="base_footprint_joint" type="fixed">
+    <parent link="base_link" />
+    <child link="base_footprint"/>
+  </joint>
+  <link name="chassis_link">
+    <inertial>
+      <mass value="${chassis_mass}"/>
+      <inertia
+        ixx="${(chassis_mass/12) * (wheelbase_width*wheelbase_width + chassis_height*chassis_height)}"
+        ixy="0.0"
+        ixz="0.0"
+        iyy="${(chassis_mass/12) * (wheelbase_length*wheelbase_length + chassis_height*chassis_height)}"
+        iyz="0.0"
+        izz="${(chassis_mass/12) * (wheelbase_length*wheelbase_length + wheelbase_width*wheelbase_width)}"/>
+      <origin xyz="0 0 0"/>
+    </inertial>
     <visual>
-        <origin xyz="0 0 0" rpy="0 0 0"/>
-        <geometry>
-            <box size="0.01 0.01 0.01"/>
-        </geometry>
+      <geometry>
+        <box size="${wheelbase_length} ${wheelbase_width} ${wheel_diameter/3}"/>
+      </geometry>
     </visual>
-    <collision>
-        <origin xyz="0 0 0" rpy="0 0 0"/>
-        <geometry>
-            <box size="0.01 0.01 0.01"/>
-        </geometry>
-    </collision>
-    <xacro:box_inertia m="0.01" w="0.01" d="0.01" h="0.01"/>
-</link>
-<joint name="${steer_joint_name}" type="revolute">
-    <parent link="base_link"/>
-    <child link="${prefix}_steer_link"/>
-    <origin xyz="${-x_reflect * wheelbase_length/2} ${(y_reflect * (wheelbase_width/2 + wheel_width/2))} ${wheelbase_height/2}" rpy="0 0 0"/>
-    <axis xyz="0 0 1"/>
-    <limit lower="-0.785" upper="0.785" effort="1000" velocity="100"/>
-    <dynamics damping="0.5" friction="0.5"/>
-</joint>
-<link name="${prefix}_link">
-    <visual>
-        <origin xyz="0 0 0" rpy="${pi/2} 0 0"/>
-        <geometry>
-            <cylinder radius="${wheel_diameter/2}" length="${wheel_width}"/>
-        </geometry>
-        <material name="Gray">
-            <color rgba="0.5 0.5 0.5 1.0"/>
-        </material>
-    </visual>
-    <collision>
-        <origin xyz="0 0 0" rpy="${pi/2} 0 0"/>
-        <geometry>
-            <cylinder radius="${wheel_diameter/2}" length="${wheel_width}"/>
-        </geometry>
-    </collision>
-    <xacro:cylinder_inertia m="0.1" r="${wheel_diameter/2}" h="${wheel_width}"/>
-</link>
-<joint name="${wheel_joint_name}" type="continuous">
-    <parent link="${prefix}_steer_link"/>
-    <child link="${prefix}_link"/>
-    <origin xyz="0 0 0" rpy="0 0 0"/>
-    <axis xyz="0 1 0"/>
-</joint>
-</xacro:macro>
-<xacro:wheel prefix="back_left_wheel" x_reflect="1" y_reflect="1" joint_name="back_left_wheel_joint"/>
-<xacro:wheel prefix="back_right_wheel" x_reflect="1" y_reflect="-1" joint_name="back_right_wheel_joint"/>
-<xacro:steering_wheel prefix="front_left_wheel" x_reflect="-1" y_reflect="1" steer_joint_name="front_left_wheel_steer_joint" wheel_joint_name="front_left_wheel_joint"/>
-<xacro:steering_wheel prefix="front_right_wheel" x_reflect="-1" y_reflect="-1" steer_joint_name="front_right_wheel_steer_joint" wheel_joint_name="front_right_wheel_joint"/>
-<!-- IMU Sensor Macro -->
-<xacro:macro name="imu_sensor">
+  </link>
+  <joint name="chassis_joint" type="fixed">
+    <parent link="base_link" />
+    <child link="chassis_link"/>
+    <origin xyz="0 0 ${wheel_diameter / 2 + (wheel_diameter/8)}"/>
+  </joint>
+  <!-- ==================== Wheel Instances ==================== -->
+  <xacro:front_wheel prefix="left" parent="base_link" x="${wheelbase_length / 2}" y="${wheelbase_width / 2 + wheel_width}" z="${wheel_diameter / 2}"/>
+  <xacro:front_wheel prefix="right" parent="base_link" x="${wheelbase_length / 2}" y="-${wheelbase_width / 2 + wheel_width}" z="${wheel_diameter / 2}"/>
+  <xacro:back_wheel prefix="left" parent="base_link" x="-${wheelbase_length / 2}" y="${wheelbase_width / 2 + wheel_width}" z="${wheel_diameter / 2}"/>
+  <xacro:back_wheel prefix="right" parent="base_link" x="-${wheelbase_length / 2}" y="-${wheelbase_width / 2 + wheel_width}" z="${wheel_diameter / 2}"/>
+  <!-- ==================== Sensors ==================== -->
+  <!-- IMU Sensor -->
   <link name="imu_link">
     <visual>
@@ -166,6 +171,12 @@
     </collision>
     <inertial>
-      <mass value="0.05"/>
-      <inertia ixx="0.01" ixy="0.0" ixz="0.0" iyy="0.01" iyz="0.0" izz="0.02"/>
+      <mass value="${imu_mass}"/>
+      <inertia
+        ixx="${(imu_mass/6) * (imu_size*imu_size)}"
+        ixy="0.0"
+        ixz="0.0"
+        iyy="${(imu_mass/6) * (imu_size*imu_size)}"
+        iyz="0.0"
+        izz="${(imu_mass/6) * (imu_size*imu_size)}"/>
       <origin xyz="0 0 0"/>
     </inertial>
@@ -174,5 +185,5 @@
     <parent link="base_link" />
     <child link="imu_link"/>
-    <origin xyz="0 0 ${wheelbase_height/2}"/>
+    <origin xyz="0 0 ${wheel_diameter / 2 + 0.05}"/>
   </joint>
   <gazebo reference="imu_link">
@@ -187,11 +198,9 @@
     </sensor>
   </gazebo>
-</xacro:macro>
-<xacro:macro name="lidar_sensor">
-<xacro:property name="LiDAR_radius" value="0.03"/>
-<link name="sllidar_base_link">
+  <!-- Lidar Sensor -->
+  <link name="sllidar_base_link">
     <visual>
       <geometry>
-        <cylinder radius="${LiDAR_radius}" length="0.05"/>
+        <cylinder radius="${Lidar_radius}" length="0.05"/>
       </geometry>
     </visual>
@@ -199,10 +208,16 @@
       <origin xyz="0 0 0" rpy="0 0 0"/>
       <geometry>
-        <cylinder radius="${LiDAR_radius}" length="0.05"/>
+        <cylinder radius="${Lidar_radius}" length="0.05"/>
       </geometry>
     </collision>
     <inertial>
-      <mass value="0.05"/>
-      <inertia ixx="0.01" ixy="0.0" ixz="0.0" iyy="0.01" iyz="0.0" izz="0.02"/>
+      <mass value="${lidar_mass}"/>
+      <inertia
+        ixx="${(lidar_mass/12) * (3*Lidar_radius*Lidar_radius + lidar_height*lidar_height)}"
+        ixy="0.0"
+        ixz="0.0"
+        iyy="${(lidar_mass/12) * (3*Lidar_radius*Lidar_radius + lidar_height*lidar_height)}"
+        iyz="0.0"
+        izz="${(lidar_mass/2) * (Lidar_radius*Lidar_radius)}"/>
       <origin xyz="0 0 0"/>
     </inertial>
@@ -211,5 +226,5 @@
     <parent link="base_link" />
     <child link="sllidar_base_link"/>
-    <origin xyz="${wheelbase_length / 2} 0 ${wheel_diameter / 2 + 0.05}"/>
+    <origin xyz="${wheelbase_length / 2 - Lidar_radius} 0 ${wheel_diameter / 2 + 0.05}"/>
   </joint>
   <gazebo reference="sllidar_base_link">
@@ -238,14 +253,9 @@
           <frame_name>sllidar_base_link</frame_name>
       </plugin>
-    </sensor>
+  </sensor>
   </gazebo>
-</xacro:macro>
-<!-- Include the sensors -->
-<xacro:imu_sensor/>
-<xacro:lidar_sensor/>
-<!-- Car Gazebo Plugin -->
-<gazebo>
-  <plugin name="car_gazebo_plugin" filename="libcar_gazebo_plugin.so">
-  </plugin>
-</gazebo>
+  <!-- ==================== Gazebo Plugins ==================== -->
+  <gazebo>
+    <plugin name="car_gazebo_plugin" filename="libcar_gazebo_plugin.so"></plugin>
+  </gazebo>
 </robot>
